File: MiteOut1.kicad_sch (KiCad schematic)
At the start: 26 parts, among them J3 Conn_02x15_Counter_Clockwise, Q1 PMOS, SW2 SW_SPST

Commit message: added SD and wifi support
Parts:
- removed D1: LED, LED_THT:LED_D1.8mm_W1.8mm_H2.4mm_Horizontal_O1.27mm_Z1.6mm, symbol Device:LED
- removed R1: R, Resistor_THT:R_Axial_DIN0204_L3.6mm_D1.6mm_P5.08mm_Horizontal, symbol Device:R
Changed lines of the file:
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@@
 	(wire
 		(pts
-			(xy 85.09 130.81) (xy 73.66 130.81)
+			(xy 74.93 66.04) (xy 107.95 66.04)
 		)
 		(stroke
@@
 	(wire
 		(pts
-			(xy 74.93 66.04) (xy 107.95 66.04)
+			(xy 168.91 154.94) (xy 171.45 154.94)
 		)
 		(stroke
@@
 	(wire
 		(pts
-			(xy 168.91 154.94) (xy 171.45 154.94)
+			(xy 87.63 38.1) (xy 111.76 38.1)
 		)
 		(stroke
@@
 	(wire
 		(pts
-			(xy 73.66 76.2) (xy 107.95 76.2)
+			(xy 107.95 152.4) (xy 151.13 152.4)
 		)
 		(stroke
@@
 	(wire
 		(pts
-			(xy 87.63 38.1) (xy 111.76 38.1)
+			(xy 214.63 77.47) (xy 204.47 77.47)
 		)
 		(stroke
@@
 	(wire
 		(pts
-			(xy 107.95 152.4) (xy 151.13 152.4)
+			(xy 165.1 38.1) (xy 207.01 38.1)
 		)
 		(stroke
@@
 	(wire
 		(pts
-			(xy 214.63 77.47) (xy 204.47 77.47)
+			(xy 87.63 93.98) (xy 87.63 38.1)
 		)
 		(stroke
@@
 	(wire
 		(pts
-			(xy 165.1 38.1) (xy 207.01 38.1)
+			(xy 109.22 31.75) (xy 109.22 60.96)
 		)
 		(stroke
@@
 	(wire
 		(pts
-			(xy 87.63 93.98) (xy 87.63 38.1)
+			(xy 184.15 78.74) (xy 184.15 87.63)
 		)
 		(stroke
@@
 	(wire
 		(pts
-			(xy 109.22 31.75) (xy 109.22 60.96)
+			(xy 232.41 107.95) (xy 251.46 107.95)
 		)
 		(stroke
@@
 	(wire
 		(pts
-			(xy 184.15 78.74) (xy 184.15 87.63)
+			(xy 120.65 99.06) (xy 121.92 99.06)
 		)
 		(stroke
@@
 	(wire
 		(pts
-			(xy 232.41 107.95) (xy 251.46 107.95)
+			(xy 19.05 137.16) (xy 20.32 137.16)
 		)
 		(stroke
@@
 	(wire
 		(pts
-			(xy 120.65 99.06) (xy 121.92 99.06)
+			(xy 219.71 49.53) (xy 219.71 69.85)
 		)
 		(stroke
@@
 	(wire
 		(pts
-			(xy 19.05 137.16) (xy 20.32 137.16)
+			(xy 30.48 97.79) (xy 30.48 85.09)
 		)
 		(stroke
@@
 	(wire
 		(pts
-			(xy 219.71 49.53) (xy 219.71 69.85)
+			(xy 20.32 167.64) (xy 20.32 137.16)
 		)
 		(stroke
@@
 	(wire
 		(pts
-			(xy 30.48 97.79) (xy 30.48 85.09)
+			(xy 72.39 71.12) (xy 107.95 71.12)
 		)
 		(stroke
@@
 	(wire
 		(pts
-			(xy 20.32 167.64) (xy 20.32 137.16)
+			(xy 17.78 17.78) (xy 17.78 76.2)
 		)
 		(stroke
@@
 	(wire
 		(pts
-			(xy 72.39 71.12) (xy 107.95 71.12)
+			(xy 31.75 128.27) (xy 31.75 115.57)
 		)
 		(stroke
@@
 	(wire
 		(pts
-			(xy 17.78 17.78) (xy 17.78 76.2)
+			(xy 17.78 76.2) (xy 17.78 109.22)
 		)
 		(stroke
@@
 	(wire
 		(pts
-			(xy 31.75 128.27) (xy 31.75 115.57)
+			(xy 190.5 62.23) (xy 191.77 62.23)
 		)
 		(stroke
@@
 	(wire
 		(pts
-			(xy 17.78 76.2) (xy 17.78 109.22)
+			(xy 81.28 58.42) (xy 81.28 91.44)
 		)
 		(stroke
@@
 	(wire
 		(pts
-			(xy 190.5 62.23) (xy 191.77 62.23)
+			(xy 184.15 78.74) (xy 207.01 78.74)
 		)
 		(stroke
@@
 	(wire
 		(pts
-			(xy 81.28 58.42) (xy 81.28 91.44)
+			(xy 186.69 76.2) (xy 186.69 77.47)
 		)
 		(stroke
@@
 	(wire
 		(pts
-			(xy 184.15 78.74) (xy 207.01 78.74)
+			(xy 186.69 77.47) (xy 186.69 83.82)
 		)
 		(stroke
@@
 	(wire
 		(pts
-			(xy 73.66 130.81) (xy 73.66 76.2)
+			(xy 66.04 68.58) (xy 107.95 68.58)
 		)
 		(stroke
@@
 		)
 	)
-	(wire
-		(pts
-			(xy 186.69 76.2) (xy 186.69 77.47)
-		)
-		(stroke
-			(width 0)
-			(type default)
-		)
-	)
-	(wire
-		(pts
-			(xy 186.69 77.47) (xy 186.69 83.82)
-		)
-		(stroke
-			(width 0)
-			(type default)
-		)
-	)
-	(wire
-		(pts
-			(xy 66.04 68.58) (xy 107.95 68.58)
-		)
-		(stroke
-			(width 0)
-			(type default)
-		)
-	)
 	(symbol
 		(lib_id "Miteout1:VCC_sens")
@@
 				(path "/5a6f6220-e177-4946-83ab-218a165d7855"
 					(reference "#PWR016")
-					(unit 1)
-				)
-			)
-		)
-	)
-	(symbol
-		(lib_id "Device:LED")
-		(at 85.09 127 270)
-		(unit 1)
-		(exclude_from_sim no)
-		(in_bom yes)
-		(on_board yes)
-		(dnp no)
-		(fields_autoplaced yes)
-		(property "Reference" "D1"
-			(at 87.63 124.1424 90)
-			(effects
-				(font
-					(size 1.27 1.27)
-				)
-				(justify left)
-			)
-		)
-		(property "Value" "LED"
-			(at 87.63 126.6824 90)
-			(effects
-				(font
-					(size 1.27 1.27)
-				)
-				(justify left)
-			)
-		)
-		(property "Footprint" "LED_THT:LED_D1.8mm_W1.8mm_H2.4mm_Horizontal_O1.27mm_Z1.6mm"
-			(at 85.09 127 0)
-			(effects
-				(font
-					(size 1.27 1.27)
-				)
-				(hide yes)
-			)
-		)
-		(property "Datasheet" "~"
-			(at 85.09 127 0)
-			(effects
-				(font
-					(size 1.27 1.27)
-				)
-				(hide yes)
-			)
-		)
-		(property "Description" "Light emitting diode"
-			(at 85.09 127 0)
-			(effects
-				(font
-					(size 1.27 1.27)
-				)
-				(hide yes)
-			)
-		)
-		(property "Sim.Pins" "1=K 2=A"
-			(at 85.09 127 0)
-			(effects
-				(font
-					(size 1.27 1.27)
-				)
-				(hide yes)
-			)
-		)
-		(pin "1"
-		)
-		(pin "2"
-		)
-		(instances
-			(project ""
-				(path "/5a6f6220-e177-4946-83ab-218a165d7855"
-					(reference "D1")
 					(unit 1)
 				)
@@
 	(symbol
 		(lib_id "power:GND")
-		(at 85.09 115.57 180)
-		(unit 1)
-		(exclude_from_sim no)
-		(in_bom yes)
-		(on_board yes)
-		(dnp no)
-		(fields_autoplaced yes)
-		(property "Reference" "#PWR02"
-			(at 85.09 109.22 0)
-			(effects
-				(font
-					(size 1.27 1.27)
-				)
-				(hide yes)
-			)
-		)
-		(property "Value" "GND"
-			(at 85.09 110.49 0)
-			(effects
-				(font
-					(size 1.27 1.27)
-				)
-			)
-		)
-		(property "Footprint" ""
-			(at 85.09 115.57 0)
-			(effects
-				(font
-					(size 1.27 1.27)
-				)
-				(hide yes)
-			)
-		)
-		(property "Datasheet" ""
-			(at 85.09 115.57 0)
-			(effects
-				(font
-					(size 1.27 1.27)
-				)
-				(hide yes)
-			)
-		)
-		(property "Description" "Power symbol creates a global label with name \"GND\" , ground"
-			(at 85.09 115.57 0)
-			(effects
-				(font
-					(size 1.27 1.27)
-				)
-				(hide yes)
-			)
-		)
-		(pin "1"
-		)
-		(instances
-			(project ""
-				(path "/5a6f6220-e177-4946-83ab-218a165d7855"
-					(reference "#PWR02")
-					(unit 1)
-				)
-			)
-		)
-	)
-	(symbol
-		(lib_id "power:GND")
 		(at 172.72 146.05 90)
 		(unit 1)
@@
 					(unit 1)
 				)
-			)
-		)
-	)
-	(symbol
-		(lib_id "Device:R")
-		(at 85.09 119.38 0)
-		(unit 1)
-		(exclude_from_sim no)
-		(in_bom yes)
-		(on_board yes)
-		(dnp no)
-		(fields_autoplaced yes)
-		(property "Reference" "R1"
-			(at 87.63 118.1099 0)
-			(effects
-				(font
-					(size 1.27 1.27)
-				)
-				(justify left)
-			)
-		)
-		(property "Value" "R"
-			(at 87.63 120.6499 0)
-			(effects
-				(font
-					(size 1.27 1.27)
-				)
-				(justify left)
-			)
-		)
-		(property "Footprint" "Resistor_THT:R_Axial_DIN0204_L3.6mm_D1.6mm_P5.08mm_Horizontal"
-			(at 83.312 119.38 90)
-			(effects
-				(font
-					(size 1.27 1.27)
-				)
-				(hide yes)
-			)
-		)
-		(property "Datasheet" "~"
-			(at 85.09 119.38 0)
-			(effects
-				(font
-					(size 1.27 1.27)
-				)
-				(hide yes)
-			)
-		)
-		(property "Description" "Resistor"
-			(at 85.09 119.38 0)
-			(effects
-				(font
-					(size 1.27 1.27)
-				)
-				(hide yes)
-			)
-		)
-		(pin "2"
-		)
-		(pin "1"
-		)
-		(instances
-			(project ""
-				(path "/5a6f6220-e177-4946-83ab-218a165d7855"
-					(reference "R1")
-					(unit 1)
-				)
