File: pcb/MiteOut1-2026-01-06_230634/MiteOut1.kicad_sch (KiCad schematic)
At the start: 18 parts, among them J3 Conn_02x15_Counter_Clockwise, Q1 PMOS, SW2 SW_SPST

Commit message: ERC
Parts:
- Clock: value ~ -> Clock
Connections:
- net GND: now also BQ1.5 (Ground); no longer BME4.3 (Pin_3), BQ1. (EN), J3.14 (Pin_14)
- net at H11.MP: now also BQ1.1 (Solar_in); no longer BQ1. (EN)
- net at SW2.2 (B): now also BQ1.7 (5v); no longer BQ1. (EN)
- no-connect marks 14 -> 17
Changed lines of the file:
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@@
+	)
+	(no_connect
+		(at 107.95 68.58)
 	)
 	(no_connect
@@
 	)
 	(no_connect
+		(at 228.6 134.62)
+	)
+	(no_connect
 		(at 107.95 76.2)
+	)
+	(no_connect
+		(at 107.95 71.12)
 	)
 	(no_connect
@@
 	(wire
 		(pts
-			(xy 227.33 58.42) (xy 240.03 58.42)
+			(xy 226.06 58.42) (xy 240.03 58.42)
 		)
 		(stroke
@@
 	(wire
 		(pts
+			(xy 204.47 34.29) (xy 204.47 30.48)
+		)
+		(stroke
+			(width 0)
+			(type default)
+		)
+	)
+	(wire
+		(pts
 			(xy 107.95 123.19) (xy 107.95 158.75)
 		)
@@
 	(wire
 		(pts
-			(xy 189.23 57.15) (xy 189.23 58.42)
-		)
-		(stroke
-			(width 0)
-			(type default)
-		)
-	)
-	(wire
-		(pts
 			(xy 172.72 139.7) (xy 172.72 171.45)
 		)
@@
 	(wire
 		(pts
+			(xy 245.11 35.56) (xy 245.11 31.75)
+		)
+		(stroke
+			(width 0)
+			(type default)
+		)
+	)
+	(wire
+		(pts
 			(xy 87.63 93.98) (xy 87.63 38.1)
 		)
@@
 		(pts
 			(xy 81.28 39.37) (xy 81.28 91.44)
+		)
+		(stroke
+			(width 0)
+			(type default)
+		)
+	)
+	(wire
+		(pts
+			(xy 242.57 33.02) (xy 242.57 31.75)
 		)
 		(stroke
@@
 	)
 	(label "Sensor VCC"
-		(at 189.23 58.42 270)
+		(at 189.23 57.15 270)
 		(effects
 			(font
@@
 	)
 	(label "Sensor VCC"
-		(at 245.11 31.75 270)
+		(at 245.11 35.56 270)
 		(effects
 			(font
@@
 	)
 	(label "Sensor VCC"
-		(at 204.47 30.48 270)
+		(at 204.47 34.29 270)
 		(effects
 			(font
@@
 	)
 	(symbol
+		(lib_name "GND_2")
+		(lib_id "power:GND")
+		(at 242.57 33.02 0)
+		(unit 1)
+		(exclude_from_sim no)
+		(in_bom yes)
+		(on_board yes)
+		(dnp no)
+		(fields_autoplaced yes)
+		(property "Reference" "#PWR02"
+			(at 242.57 39.37 0)
+			(effects
+				(font
+					(size 1.27 1.27)
+				)
+				(hide yes)
+			)
+		)
+		(property "Value" "GND"
+			(at 242.57 38.1 0)
+			(effects
+				(font
+					(size 1.27 1.27)
+				)
+			)
+		)
+		(property "Footprint" ""
+			(at 242.57 33.02 0)
+			(effects
+				(font
+					(size 1.27 1.27)
+				)
+				(hide yes)
+			)
+		)
+		(property "Datasheet" ""
+			(at 242.57 33.02 0)
+			(effects
+				(font
+					(size 1.27 1.27)
+				)
+				(hide yes)
+			)
+		)
+		(property "Description" "Power symbol creates a global label with name \"GND\" , ground"
+			(at 242.57 33.02 0)
+			(effects
+				(font
+					(size 1.27 1.27)
+				)
+				(hide yes)
+			)
+		)
+		(pin "1"
+		)
+		(instances
+			(project "MiteOut1"
+				(path "/5a6f6220-e177-4946-83ab-218a165d7855"
+					(reference "#PWR02")
+					(unit 1)
+				)
+			)
+		)
+	)
+	(symbol
+		(lib_name "MountingHole_Pad_MP_1")
 		(lib_id "Mechanical:MountingHole_Pad_MP")
 		(at 215.9 115.57 90)
@@
 			)
 		)
-		(property "Value" "~"
+		(property "Value" "Clock"
 			(at 198.12 50.8 90)
 			(effects
@@
 	)
 	(symbol
+		(lib_name "MountingHole_Pad_MP_3")
 		(lib_id "Mechanical:MountingHole_Pad_MP")
-		(at 224.79 58.42 90)
+		(at 223.52 58.42 90)
 		(unit 1)
 		(exclude_from_sim no)
@@
 		(fields_autoplaced yes)
 		(property "Reference" "H4"
-			(at 222.2499 55.88 0)
+			(at 217.678 62.484 0)
 			(effects
 				(font
@@
 		)
 		(property "Value" "LoadCell2"
-			(at 223.52 54.61 90)
+			(at 222.758 51.562 90)
 			(effects
 				(font
@@
 		)
 		(property "Footprint" "MiteOut:throughole"
-			(at 224.79 58.42 0)
+			(at 214.63 58.166 0)
 			(effects
 				(font
@@
 		)
 		(property "Datasheet" "~"
-			(at 224.79 58.42 0)
+			(at 223.52 58.42 0)
 			(effects
 				(font
@@
 		)
 		(property "Description" "Mounting Hole with connection as pad named MP"
-			(at 224.79 58.42 0)
+			(at 212.344 59.182 0)
 			(effects
 				(font
@@
 	)
 	(symbol
+		(lib_name "Conn_01x04_1")
 		(lib_id "Connector_Generic:Conn_01x04")
 		(at 199.39 25.4 90)
@@
 	)
 	(symbol
+		(lib_name "MountingHole_Pad_MP_2")
 		(lib_id "Mechanical:MountingHole_Pad_MP")
 		(at 231.14 55.88 90)
@@
 	)
 	(symbol
+		(lib_name "GND_1")
 		(lib_id "power:GND")
 		(at 91.44 99.06 270)
@@
 	)
 	(symbol
+		(lib_name "MountingHole_Pad_MP_5")
 		(lib_id "Mechanical:MountingHole_Pad_MP")
 		(at 214.63 63.5 90)
@@
 			)
 		)
-		(pin ""
-		)
-		(pin ""
-		)
-		(pin ""
-		)
-		(pin ""
-		)
-		(pin ""
-		)
-		(pin ""
-		)
-		(pin ""
-		)
-		(pin ""
+		(pin "5"
+		)
+		(pin "6"
+		)
+		(pin "2"
+		)
+		(pin "7"
+		)
+		(pin "8"
+		)
+		(pin "1"
+		)
+		(pin "3"
+		)
+		(pin "4"
 		)
 		(instances
@@
 	)
 	(symbol
+		(lib_name "MountingHole_Pad_MP_4")
 		(lib_id "Mechanical:MountingHole_Pad_MP")
 		(at 219.71 60.96 90)
@@
 					(unit 1)
 				)
-			)
-		)
-	)
-	(symbol
-		(lib_id "power:GND")
-		(at 242.57 31.75 0)
-		(unit 1)
-		(exclude_from_sim no)
-		(in_bom yes)
-		(on_board yes)
-		(dnp no)
-		(fields_autoplaced yes)
-		(property "Reference" "#PWR02"
-			(at 242.57 38.1 0)
-			(effects
-				(font
-					(size 1.27 1.27)
-				)
-				(hide yes)
-			)
-		)
-		(property "Value" "GND"
-			(at 242.57 36.83 0)
-			(effects
-				(font
-					(size 1.27 1.27)
-				)
-			)
-		)
-		(property "Footprint" ""
-			(at 242.57 31.75 0)
-			(effects
-				(font
-					(size 1.27 1.27)
-				)
-				(hide yes)
-			)
-		)
-		(property "Datasheet" ""
-			(at 242.57 31.75 0)
-			(effects
-				(font
-					(size 1.27 1.27)
-				)
-				(hide yes)
-			)
-		)
-		(property "Description" "Power symbol creates a global label with name \"GND\" , ground"
-			(at 242.57 31.75 0)
-			(effects
-				(font
-					(size 1.27 1.27)
-				)
-				(hide yes)
-			)
-		)
-		(pin "1"
-		)
-		(instances
-			(project "MiteOut1"
-				(path "/5a6f6220-e177-4946-83ab-218a165d7855"
-					(reference "#PWR02")
-					(unit 1)
-				)

Commit message: going to bed before the 10a
Parts:
- BME1, BME2, BME3, BME4: footprint Connector_JST:JST_EH_B4B-EH-A_1x04_P2.50mm_Vertical -> MiteOut1:4Wire
- Clock1: renamed from Clock; footprint (none) -> MiteOut1:4Wire
