File: pcb/MiteOut1-2026-01-06_230634/MiteOut1.kicad_pcb (KiCad board)
At the start: 2 copper layers, 81 x 73 mm, 19 parts, among them J3 Conn_02x15_Counter_Clockwise, Q1 PMOS, SW2 SW_SPST

Commit message: going to bed before the 10a
Parts:
- added BME2: Conn_01x04, MiteOut1:4Wire, F.Cu at (47.2, 69.8)
- added BME3: Conn_01x04, MiteOut1:4Wire, F.Cu at (47.2, 76.5)
- added BME4: Conn_01x04, MiteOut1:4Wire, F.Cu at (47.2, 83.2)
- added Clock1: Clock, MiteOut1:4Wire, F.Cu at (47.2, 90.0)
- BME1: renamed from StemmaQT1; footprint Connector_JST:JST_EH_B4B-EH-A_1x04_P2.50mm_Vertical -> MiteOut1:4Wire
- U1: footprint MiteOut:Clock -> MiteOut1:4Wire
- moved U1 18.2 mm to (62.0, 68.9), turned to 0 degrees
- moved BME1 8.02 mm to (74.4, 125.6)
Connections:
- BME1 pad 1: GND -> /Wire0 SDA
- BME1 pad 2: Net-(HX711-VCC) -> /Wire0 SCK
- BME1 pad 3: Net-(HX711-DT) -> GND
- BME1 pad 4: Net-(HX711-SCK) -> /Sensor VCC
- BQ1 pad 6: Net-(BQ1-Bat_Voltage) -> unconnected-(BQ1-Bat_Voltage-Pad6)
- HX711 pad 10: Net-(HX711-VCC) -> /Sensor VCC
- HX711 pad 8: Net-(HX711-DT) -> /HX711 DT
- HX711 pad 9: Net-(HX711-SCK) -> /HX711 CLK
- INO1 pad 1: Net-(INO1-VCC) -> /Sensor VCC
- INO1 pad 3: Net-(HX711-SCK) -> /Wire0 SCK
- INO1 pad 4: Net-(HX711-DT) -> /Wire0 SDA
- INO1 pad 7: Net-(BQ1-Bat_Voltage) -> Net-(INO1-VIN+)
- INO1 pad 8: +5V -> /Sensor VCC
- J3 pad 14: GND -> Net-(J3-Pin_14)
- J3 pad 15: +5V -> Net-(J3-Pin_15)
- J3 pad 26: Net-(HX711-DT) -> /Wire0 SCK
- J3 pad 29: Net-(HX711-SCK) -> /Wire0 SDA
- J3 pad 4: unconnected-(J3-Pin_4-Pad4) -> Net-(J3-Pin_4)
- J3 pad 6: unconnected-(J3-Pin_6-Pad6) -> /Wire1 SCK
- J3 pad 7: unconnected-(J3-Pin_7-Pad7) -> /Wire1 SCK
- J3 pad 8: unconnected-(J3-Pin_8-Pad8) -> /HX711 DT
- J3 pad 9: unconnected-(J3-Pin_9-Pad9) -> /HX711 CLK
- Q1 pad D: unconnected-(Q1-PadD) -> (no net)
- Q1 pad G: unconnected-(Q1-PadG) -> (no net)
- Q1 pad S: +5V -> (no net)
- SW2 pad 1: +5V -> Net-(J3-Pin_15)
- U3 pad 8: Net-(HX711-VCC) -> (no net)
Routing:
- net Net-(HX711-VCC): track 114.5 -> 0.00 mm, vias 2 -> 0
- net /Sensor VCC: track 0.00 -> 114.5 mm, vias 0 -> 2
- net (no net): track 60.5 -> 164.4 mm, vias 1 -> 3
- net +5V: track 95.0 -> 0.00 mm, vias 1 -> 0
- net Net-(J3-Pin_4): track 0.00 -> 60.5 mm, vias 0 -> 1
- net Net-(BQ1-Bat_Voltage): track 50.0 -> 0.00 mm, vias 2 -> 0
- net unconnected-(J3-Pin_6-Pad6): track 43.0 -> 0.00 mm, vias 1 -> 0
- net /Wire1 SCK: track 0.00 -> 43.0 mm, vias 0 -> 1
- net Net-(J3-Pin_2): track 11.9 -> 0.00 mm
- net Net-(J3-Pin_6): track 7.47 -> 0.00 mm

Commit message: pcb changes
Parts:
- removed U1: ~, MiteOut1:4Wire
- added G***: LOGO, MiteOut1:MiteOutLogoHex, F.Cu at (118.9, 118.8)
- moved Q1 61.0 mm to (56.5, 64.0)
- moved BME3 60.7 mm to (74.6, 130.6)
- moved BME1 60.1 mm to (73.7, 65.5)
- moved BME2 56.2 mm to (62.5, 123.9)
- moved BME4 49.7 mm to (62.5, 130.5)
- moved Clock1 43.6 mm to (74.6, 123.9)
- moved SW2 36.4 mm to (69.8, 71.5)
- moved G*** 36.4 mm to (102.1, 151.9)
Routing:
- net (no net): track 164.4 -> 0.00 mm, vias 3 -> 0
- net GND: track 118.2 -> 0.00 mm, vias 8 -> 0
- net /Sensor VCC: track 114.5 -> 0.00 mm, vias 2 -> 0
- net Net-(HX711-SCK): track 94.3 -> 0.00 mm, vias 3 -> 0
- net Net-(HX711-DT): track 91.0 -> 0.00 mm, vias 4 -> 0
- net Net-(J3-Pin_4): track 60.5 -> 0.00 mm, vias 1 -> 0
- net Net-(J3-Pin_18): track 53.8 -> 0.00 mm, vias 1 -> 0
- net unconnected-(J3-Pin_3-Pad3): track 49.5 -> 0.00 mm, vias 1 -> 0
- net unconnected-(J3-Pin_2-Pad2): track 49.1 -> 0.00 mm, vias 1 -> 0
- net /Wire1 SCK: track 43.0 -> 0.00 mm, vias 1 -> 0
- net Net-(BQ1-5v): track 33.3 -> 0.00 mm, vias 1 -> 0
- net Net-(HX711-A+): track 32.5 -> 0.00 mm
- net Net-(HX711-A-): track 28.3 -> 0.00 mm
- net Net-(J3-Pin_13): track 25.6 -> 0.00 mm
- net Net-(HX711-E-): track 24.2 -> 0.00 mm
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Other:
- board text added: "DATA UNIT V1.2"
- board text removed: "DATA UNIT V1.1"
- board text removed: "GND 5V 5V"
- board text removed: "GND 5V SDA SCL"
- board text removed: "Real Time Clock"
- board text removed: "SCL SDA 3V3"
- board text removed: "\/ Battery \/"
